Commit message: fix: urdf base_link as root, headless launch arg, bridge qos hints

File: workspace/src/maze_worlds/urdf/maze_bot.urdf.xacro (robot description, xacro)
@@ -27,5 +27,4 @@
     </inertial>
   </xacro:macro>
-  <link name="base_footprint"/>
   <link name="base_link">
     <visual>
@@ -38,9 +37,4 @@
     <xacro:box_inertia m="2.0" x="${base_l}" y="${base_w}" z="${base_h}"/>
   </link>
-  <joint name="base_joint" type="fixed">
-    <parent link="base_footprint"/>
-    <child link="base_link"/>
-    <origin xyz="0 0 ${wheel_r + base_h/2}"/>
-  </joint>
   <!-- wheels -->
   <xacro:macro name="wheel" params="prefix y_offset">
